Commit message: Remove duplicate xacro pi property

File: src/diffbot_gazebo/urdf/diffbot.urdf.xacro (robot description, xacro)
@@ -10,5 +10,4 @@
   <xacro:property name="wheel_z" value="0.085"/>
   <xacro:property name="caster_radius" value="0.035"/>
-  <xacro:property name="pi" value="3.141592653589793"/>
   <material name="body_blue"><color rgba="0.05 0.22 0.55 1"/></material>
   <material name="top_silver"><color rgba="0.75 0.8 0.86 1"/></material>

Commit message: Improve robot model and teleop feedback

File: src/diffbot_gazebo/urdf/diffbot.urdf.xacro (robot description, xacro)
@@ -3,5 +3,5 @@
   <xacro:property name="base_length" value="0.46"/>
   <xacro:property name="base_width" value="0.32"/>
-  <xacro:property name="base_height" value="0.12"/>
+  <xacro:property name="base_height" value="0.18"/>
   <xacro:property name="wheel_radius" value="0.085"/>
   <xacro:property name="wheel_width" value="0.045"/>
@@ -16,4 +16,6 @@
   <material name="accent_orange"><color rgba="1.0 0.45 0.08 1"/></material>
   <material name="sensor_glass"><color rgba="0.02 0.08 0.12 0.75"/></material>
+  <material name="lidar_dark"><color rgba="0.01 0.015 0.02 1"/></material>
+  <material name="lidar_blue"><color rgba="0.1 0.75 0.95 0.85"/></material>
   <link name="base_footprint"/>
   <joint name="base_footprint_joint" type="fixed">
@@ -40,4 +42,19 @@
       <material name="top_silver"/>
     </visual>
+    <visual name="upper_shell">
+      <origin xyz="-0.03 0 ${base_height / 2.0 + 0.055}"/>
+      <geometry><box size="0.28 0.20 0.07"/></geometry>
+      <material name="body_blue"/>
+    </visual>
+    <visual name="orange_side_left">
+      <origin xyz="-0.02 ${base_width / 2.0 + 0.006} 0.015"/>
+      <geometry><box size="0.30 0.012 0.035"/></geometry>
+      <material name="accent_orange"/>
+    </visual>
+    <visual name="orange_side_right">
+      <origin xyz="-0.02 ${-base_width / 2.0 - 0.006} 0.015"/>
+      <geometry><box size="0.30 0.012 0.035"/></geometry>
+      <material name="accent_orange"/>
+    </visual>
     <visual name="front_bumper">
       <origin xyz="${base_length / 2.0 + 0.018} 0 -0.015"/>
@@ -131,4 +148,27 @@
     <origin xyz="0.18 0 -0.06" rpy="0 0 0"/>
   </joint>
+  <link name="rear_caster_link">
+    <inertial>
+      <mass value="0.12"/>
+      <inertia ixx="0.00015" ixy="0" ixz="0" iyy="0.00015" iyz="0" izz="0.00015"/>
+    </inertial>
+    <collision>
+      <geometry><sphere radius="${caster_radius}"/></geometry>
+      <surface>
+        <friction>
+          <ode><mu>0.01</mu><mu2>0.01</mu2></ode>
+        </friction>
+      </surface>
+    </collision>
+    <visual>
+      <geometry><sphere radius="${caster_radius}"/></geometry>
+      <material name="rim_gray"/>
+    </visual>
+  </link>
+  <joint name="rear_caster_joint" type="fixed">
+    <parent link="base_link"/>
+    <child link="rear_caster_link"/>
+    <origin xyz="-0.18 0 -0.06" rpy="0 0 0"/>
+  </joint>
   <link name="sensor_mast_link">
     <collision>
@@ -151,4 +191,34 @@
     <child link="sensor_mast_link"/>
     <origin xyz="0.08 0 ${base_height / 2.0 + 0.015}" rpy="0 0 0"/>
+  </joint>
+  <link name="lidar_link">
+    <inertial>
+      <mass value="0.18"/>
+      <inertia ixx="0.00025" ixy="0" ixz="0" iyy="0.00025" iyz="0" izz="0.00035"/>
+    </inertial>
+    <collision>
+      <origin xyz="0 0 0.025"/>
+      <geometry><cylinder radius="0.055" length="0.05"/></geometry>
+    </collision>
+    <visual name="lidar_base">
+      <origin xyz="0 0 0.018"/>
+      <geometry><cylinder radius="0.06" length="0.036"/></geometry>
+      <material name="lidar_dark"/>
+    </visual>
+    <visual name="lidar_scan_band">
+      <origin xyz="0 0 0.045"/>
+      <geometry><cylinder radius="0.052" length="0.022"/></geometry>
+      <material name="lidar_blue"/>
+    </visual>
+    <visual name="lidar_cap">
+      <origin xyz="0 0 0.064"/>
+      <geometry><cylinder radius="0.045" length="0.016"/></geometry>
+      <material name="lidar_dark"/>
+    </visual>
+  </link>
+  <joint name="lidar_joint" type="fixed">
+    <parent link="base_link"/>
+    <child link="lidar_link"/>
+    <origin xyz="-0.08 0 ${base_height / 2.0 + 0.095}" rpy="0 0 0"/>
   </joint>
   <gazebo reference="base_link">

Commit message: Lower caster supports for balance

File: src/diffbot_gazebo/urdf/diffbot.urdf.xacro (robot description, xacro)
@@ -10,4 +10,5 @@
   <xacro:property name="wheel_z" value="0.085"/>
   <xacro:property name="caster_radius" value="0.035"/>
+  <xacro:property name="caster_z" value="${-base_height / 2.0}"/>
   <material name="body_blue"><color rgba="0.05 0.22 0.55 1"/></material>
   <material name="top_silver"><color rgba="0.75 0.8 0.86 1"/></material>
@@ -146,5 +147,5 @@
     <parent link="base_link"/>
     <child link="front_caster_link"/>
-    <origin xyz="0.18 0 -0.06" rpy="0 0 0"/>
+    <origin xyz="0.18 0 ${caster_z}" rpy="0 0 0"/>
   </joint>
   <link name="rear_caster_link">
@@ -169,5 +170,5 @@
     <parent link="base_link"/>
     <child link="rear_caster_link"/>
-    <origin xyz="-0.18 0 -0.06" rpy="0 0 0"/>
+    <origin xyz="-0.20 0 ${caster_z}" rpy="0 0 0"/>
   </joint>
   <link name="sensor_mast_link">

Commit message: Reduce caster friction

File: src/diffbot_gazebo/urdf/diffbot.urdf.xacro (robot description, xacro)
@@ -9,6 +9,6 @@
   <xacro:property name="wheel_x" value="0.02"/>
   <xacro:property name="wheel_z" value="0.085"/>
-  <xacro:property name="caster_radius" value="0.035"/>
-  <xacro:property name="caster_z" value="${-base_height / 2.0}"/>
+  <xacro:property name="caster_radius" value="0.025"/>
+  <xacro:property name="caster_z" value="${-base_height / 2.0 - 0.006}"/>
   <material name="body_blue"><color rgba="0.05 0.22 0.55 1"/></material>
   <material name="top_silver"><color rgba="0.75 0.8 0.86 1"/></material>
@@ -128,6 +128,6 @@
   <link name="front_caster_link">
     <inertial>
-      <mass value="0.12"/>
-      <inertia ixx="0.00015" ixy="0" ixz="0" iyy="0.00015" iyz="0" izz="0.00015"/>
+      <mass value="0.03"/>
+      <inertia ixx="0.00003" ixy="0" ixz="0" iyy="0.00003" iyz="0" izz="0.00003"/>
     </inertial>
     <collision>
@@ -135,10 +135,13 @@
       <surface>
         <friction>
-          <ode><mu>0.01</mu><mu2>0.01</mu2></ode>
+          <ode><mu>0.001</mu><mu2>0.001</mu2></ode>
         </friction>
+        <contact>
+          <ode><kp>100000</kp><kd>1</kd><max_vel>0.2</max_vel><min_depth>0.001</min_depth></ode>
+        </contact>
       </surface>
     </collision>
     <visual>
-      <geometry><sphere radius="${caster_radius}"/></geometry>
+      <geometry><sphere radius="0.035"/></geometry>
       <material name="rim_gray"/>
     </visual>
@@ -151,6 +154,6 @@
   <link name="rear_caster_link">
     <inertial>
-      <mass value="0.12"/>
-      <inertia ixx="0.00015" ixy="0" ixz="0" iyy="0.00015" iyz="0" izz="0.00015"/>
+      <mass value="0.03"/>
+      <inertia ixx="0.00003" ixy="0" ixz="0" iyy="0.00003" iyz="0" izz="0.00003"/>
     </inertial>
     <collision>
@@ -158,10 +161,13 @@
       <surface>
         <friction>
-          <ode><mu>0.01</mu><mu2>0.01</mu2></ode>
+          <ode><mu>0.001</mu><mu2>0.001</mu2></ode>
         </friction>
+        <contact>
+          <ode><kp>100000</kp><kd>1</kd><max_vel>0.2</max_vel><min_depth>0.001</min_depth></ode>
+        </contact>
       </surface>
     </collision>
     <visual>
-      <geometry><sphere radius="${caster_radius}"/></geometry>
+      <geometry><sphere radius="0.035"/></geometry>
       <material name="rim_gray"/>
     </visual>

Commit message: Make caster supports visual only

File: src/diffbot_gazebo/urdf/diffbot.urdf.xacro (robot description, xacro)
@@ -131,15 +131,4 @@
       <inertia ixx="0.00003" ixy="0" ixz="0" iyy="0.00003" iyz="0" izz="0.00003"/>
     </inertial>
-    <collision>
-      <geometry><sphere radius="${caster_radius}"/></geometry>
-      <surface>
-        <friction>
-          <ode><mu>0.001</mu><mu2>0.001</mu2></ode>
-        </friction>
-        <contact>
-          <ode><kp>100000</kp><kd>1</kd><max_vel>0.2</max_vel><min_depth>0.001</min_depth></ode>
-        </contact>
-      </surface>
-    </collision>
     <visual>
       <geometry><sphere radius="0.035"/></geometry>
@@ -157,15 +146,4 @@
       <inertia ixx="0.00003" ixy="0" ixz="0" iyy="0.00003" iyz="0" izz="0.00003"/>
     </inertial>
-    <collision>
-      <geometry><sphere radius="${caster_radius}"/></geometry>
-      <surface>
-        <friction>
-          <ode><mu>0.001</mu><mu2>0.001</mu2></ode>
-        </friction>
-        <contact>
-          <ode><kp>100000</kp><kd>1</kd><max_vel>0.2</max_vel><min_depth>0.001</min_depth></ode>
-        </contact>
-      </surface>
-    </collision>
     <visual>
       <geometry><sphere radius="0.035"/></geometry>

Commit message: Restore ultra low friction caster support

File: src/diffbot_gazebo/urdf/diffbot.urdf.xacro (robot description, xacro)
@@ -10,5 +10,6 @@
   <xacro:property name="wheel_z" value="0.085"/>
   <xacro:property name="caster_radius" value="0.025"/>
-  <xacro:property name="caster_z" value="${-base_height / 2.0 - 0.006}"/>
+  <xacro:property name="base_origin_z" value="${base_height / 2.0 + 0.035}"/>
+  <xacro:property name="caster_z" value="${caster_radius - base_origin_z + 0.001}"/>
   <material name="body_blue"><color rgba="0.05 0.22 0.55 1"/></material>
   <material name="top_silver"><color rgba="0.75 0.8 0.86 1"/></material>
@@ -23,5 +24,5 @@
     <parent link="base_footprint"/>
     <child link="base_link"/>
-    <origin xyz="0 0 ${base_height / 2.0 + 0.035}" rpy="0 0 0"/>
+    <origin xyz="0 0 ${base_origin_z}" rpy="0 0 0"/>
   </joint>
   <link name="base_link">
@@ -131,4 +132,20 @@
       <inertia ixx="0.00003" ixy="0" ixz="0" iyy="0.00003" iyz="0" izz="0.00003"/>
     </inertial>
+    <collision>
+      <geometry><sphere radius="${caster_radius}"/></geometry>
+      <surface>
+        <friction>
+          <ode>
+            <mu>0.000001</mu>
+            <mu2>0.000001</mu2>
+            <slip1>1.0</slip1>
+            <slip2>1.0</slip2>
+          </ode>
+        </friction>
+        <contact>
+          <ode><kp>80000</kp><kd>0.5</kd><max_vel>0.1</max_vel><min_depth>0.0005</min_depth></ode>
+        </contact>
+      </surface>
+    </collision>
     <visual>
       <geometry><sphere radius="0.035"/></geometry>
@@ -146,4 +163,20 @@
       <inertia ixx="0.00003" ixy="0" ixz="0" iyy="0.00003" iyz="0" izz="0.00003"/>
     </inertial>
+    <collision>
+      <geometry><sphere radius="${caster_radius}"/></geometry>
+      <surface>
+        <friction>
+          <ode>
+            <mu>0.000001</mu>
+            <mu2>0.000001</mu2>
+            <slip1>1.0</slip1>
+            <slip2>1.0</slip2>
+          </ode>
+        </friction>
+        <contact>
+          <ode><kp>80000</kp><kd>0.5</kd><max_vel>0.1</max_vel><min_depth>0.0005</min_depth></ode>
+        </contact>
+      </surface>
+    </collision>
     <visual>
       <geometry><sphere radius="0.035"/></geometry>

Commit message: Align caster collision with visual support

File: src/diffbot_gazebo/urdf/diffbot.urdf.xacro (robot description, xacro)
@@ -9,7 +9,7 @@
   <xacro:property name="wheel_x" value="0.02"/>
   <xacro:property name="wheel_z" value="0.085"/>
-  <xacro:property name="caster_radius" value="0.025"/>
+  <xacro:property name="caster_radius" value="0.035"/>
   <xacro:property name="base_origin_z" value="${base_height / 2.0 + 0.035}"/>
-  <xacro:property name="caster_z" value="${caster_radius - base_origin_z + 0.001}"/>
+  <xacro:property name="caster_z" value="${caster_radius - base_origin_z - 0.004}"/>
   <material name="body_blue"><color rgba="0.05 0.22 0.55 1"/></material>
   <material name="top_silver"><color rgba="0.75 0.8 0.86 1"/></material>
@@ -149,5 +149,5 @@
     </collision>
     <visual>
-      <geometry><sphere radius="0.035"/></geometry>
+      <geometry><sphere radius="${caster_radius}"/></geometry>
       <material name="rim_gray"/>
     </visual>
@@ -180,5 +180,5 @@
     </collision>
     <visual>
-      <geometry><sphere radius="0.035"/></geometry>
+      <geometry><sphere radius="${caster_radius}"/></geometry>
       <material name="rim_gray"/>
     </visual>

Commit message: Keep drive wheels grounded

File: src/diffbot_gazebo/urdf/diffbot.urdf.xacro (robot description, xacro)
@@ -11,5 +11,5 @@
   <xacro:property name="caster_radius" value="0.035"/>
   <xacro:property name="base_origin_z" value="${base_height / 2.0 + 0.035}"/>
-  <xacro:property name="caster_z" value="${caster_radius - base_origin_z - 0.004}"/>
+  <xacro:property name="caster_z" value="${caster_radius - base_origin_z}"/>
   <material name="body_blue"><color rgba="0.05 0.22 0.55 1"/></material>
   <material name="top_silver"><color rgba="0.75 0.8 0.86 1"/></material>

Commit message: Restore drive traction

File: src/diffbot_gazebo/urdf/diffbot.urdf.xacro (robot description, xacro)
@@ -132,4 +132,19 @@
       <inertia ixx="0.00003" ixy="0" ixz="0" iyy="0.00003" iyz="0" izz="0.00003"/>
     </inertial>
+    <visual>
+      <geometry><sphere radius="${caster_radius}"/></geometry>
+      <material name="rim_gray"/>
+    </visual>
+  </link>
+  <joint name="front_caster_joint" type="fixed">
+    <parent link="base_link"/>
+    <child link="front_caster_link"/>
+    <origin xyz="0.18 0 ${caster_z}" rpy="0 0 0"/>
+  </joint>
+  <link name="rear_caster_link">
+    <inertial>
+      <mass value="0.03"/>
+      <inertia ixx="0.00003" ixy="0" ixz="0" iyy="0.00003" iyz="0" izz="0.00003"/>
+    </inertial>
     <collision>
       <geometry><sphere radius="${caster_radius}"/></geometry>
@@ -153,35 +168,4 @@
     </visual>
   </link>
-  <joint name="front_caster_joint" type="fixed">
-    <parent link="base_link"/>
-    <child link="front_caster_link"/>
-    <origin xyz="0.18 0 ${caster_z}" rpy="0 0 0"/>
-  </joint>
-  <link name="rear_caster_link">
-    <inertial>
-      <mass value="0.03"/>
-      <inertia ixx="0.00003" ixy="0" ixz="0" iyy="0.00003" iyz="0" izz="0.00003"/>
-    </inertial>
-    <collision>
-      <geometry><sphere radius="${caster_radius}"/></geometry>
-      <surface>
-        <friction>
-          <ode>
-            <mu>0.000001</mu>
-            <mu2>0.000001</mu2>
-            <slip1>1.0</slip1>
-            <slip2>1.0</slip2>
-          </ode>
-        </friction>
-        <contact>
-          <ode><kp>80000</kp><kd>0.5</kd><max_vel>0.1</max_vel><min_depth>0.0005</min_depth></ode>
-        </contact>
-      </surface>
-    </collision>
-    <visual>
-      <geometry><sphere radius="${caster_radius}"/></geometry>
-      <material name="rim_gray"/>
-    </visual>
-  </link>
   <joint name="rear_caster_joint" type="fixed">
     <parent link="base_link"/>
@@ -245,11 +229,15 @@
   <gazebo reference="left_wheel_link">
     <material>Gazebo/Black</material>
-    <mu1>1.0</mu1>
-    <mu2>1.0</mu2>
+    <mu1>2.0</mu1>
+    <mu2>2.0</mu2>
+    <kp>1000000</kp>
+    <kd>1</kd>
   </gazebo>
   <gazebo reference="right_wheel_link">
     <material>Gazebo/Black</material>
-    <mu1>1.0</mu1>
-    <mu2>1.0</mu2>
+    <mu1>2.0</mu1>
+    <mu2>2.0</mu2>
+    <kp>1000000</kp>
+    <kd>1</kd>
   </gazebo>
   <gazebo>
@@ -265,6 +253,6 @@
       <wheel_separation>${2.0 * wheel_y}</wheel_separation>
       <wheel_diameter>${2.0 * wheel_radius}</wheel_diameter>
-      <max_wheel_torque>20</max_wheel_torque>
-      <max_wheel_acceleration>2.0</max_wheel_acceleration>
+      <max_wheel_torque>80</max_wheel_torque>
+      <max_wheel_acceleration>8.0</max_wheel_acceleration>
       <command_topic>cmd_vel</command_topic>
       <odometry_topic>odom</odometry_topic>

Commit message: Continuously publish teleop commands

File: src/diffbot_gazebo/urdf/diffbot.urdf.xacro (robot description, xacro)
@@ -11,5 +11,5 @@
   <xacro:property name="caster_radius" value="0.035"/>
   <xacro:property name="base_origin_z" value="${base_height / 2.0 + 0.035}"/>
-  <xacro:property name="caster_z" value="${caster_radius - base_origin_z}"/>
+  <xacro:property name="caster_z" value="${caster_radius - base_origin_z + 0.001}"/>
   <material name="body_blue"><color rgba="0.05 0.22 0.55 1"/></material>
   <material name="top_silver"><color rgba="0.75 0.8 0.86 1"/></material>

Commit message: Refine hidden low-friction support wheels

File: src/diffbot_gazebo/urdf/diffbot.urdf.xacro (robot description, xacro)
@@ -9,5 +9,5 @@
   <xacro:property name="wheel_x" value="0.02"/>
   <xacro:property name="wheel_z" value="0.085"/>
-  <xacro:property name="caster_radius" value="0.035"/>
+  <xacro:property name="caster_radius" value="0.024"/>
   <xacro:property name="base_origin_z" value="${base_height / 2.0 + 0.035}"/>
   <xacro:property name="caster_z" value="${caster_radius - base_origin_z + 0.001}"/>
@@ -132,19 +132,4 @@
       <inertia ixx="0.00003" ixy="0" ixz="0" iyy="0.00003" iyz="0" izz="0.00003"/>
     </inertial>
-    <visual>
-      <geometry><sphere radius="${caster_radius}"/></geometry>
-      <material name="rim_gray"/>
-    </visual>
-  </link>
-  <joint name="front_caster_joint" type="fixed">
-    <parent link="base_link"/>
-    <child link="front_caster_link"/>
-    <origin xyz="0.18 0 ${caster_z}" rpy="0 0 0"/>
-  </joint>
-  <link name="rear_caster_link">
-    <inertial>
-      <mass value="0.03"/>
-      <inertia ixx="0.00003" ixy="0" ixz="0" iyy="0.00003" iyz="0" izz="0.00003"/>
-    </inertial>
     <collision>
       <geometry><sphere radius="${caster_radius}"/></geometry>
@@ -168,8 +153,39 @@
     </visual>
   </link>
+  <joint name="front_caster_joint" type="fixed">
+    <parent link="base_link"/>
+    <child link="front_caster_link"/>
+    <origin xyz="0.19 0 ${caster_z}" rpy="0 0 0"/>
+  </joint>
+  <link name="rear_caster_link">
+    <inertial>
+      <mass value="0.03"/>
+      <inertia ixx="0.00003" ixy="0" ixz="0" iyy="0.00003" iyz="0" izz="0.00003"/>
+    </inertial>
+    <collision>
+      <geometry><sphere radius="${caster_radius}"/></geometry>
+      <surface>
+        <friction>
+          <ode>
+            <mu>0.000001</mu>
+            <mu2>0.000001</mu2>
+            <slip1>1.0</slip1>
+            <slip2>1.0</slip2>
+          </ode>
+        </friction>
+        <contact>
+          <ode><kp>80000</kp><kd>0.5</kd><max_vel>0.1</max_vel><min_depth>0.0005</min_depth></ode>
+        </contact>
+      </surface>
+    </collision>
+    <visual>
+      <geometry><sphere radius="${caster_radius}"/></geometry>
+      <material name="rim_gray"/>
+    </visual>
+  </link>
   <joint name="rear_caster_joint" type="fixed">
     <parent link="base_link"/>
     <child link="rear_caster_link"/>
-    <origin xyz="-0.20 0 ${caster_z}" rpy="0 0 0"/>
+    <origin xyz="-0.19 0 ${caster_z}" rpy="0 0 0"/>
   </joint>
   <link name="sensor_mast_link">

Commit message: Remove support casters for motion test

File: src/diffbot_gazebo/urdf/diffbot.urdf.xacro (robot description, xacro)
@@ -9,7 +9,5 @@
   <xacro:property name="wheel_x" value="0.02"/>
   <xacro:property name="wheel_z" value="0.085"/>
-  <xacro:property name="caster_radius" value="0.024"/>
   <xacro:property name="base_origin_z" value="${base_height / 2.0 + 0.035}"/>
-  <xacro:property name="caster_z" value="${caster_radius - base_origin_z + 0.001}"/>
   <material name="body_blue"><color rgba="0.05 0.22 0.55 1"/></material>
   <material name="top_silver"><color rgba="0.75 0.8 0.86 1"/></material>
@@ -126,66 +124,4 @@
     <origin xyz="${wheel_x} ${-wheel_y} ${-base_height / 2.0 + wheel_z - 0.035}" rpy="0 0 0"/>
     <axis xyz="0 1 0"/>
-  </joint>
-  <link name="front_caster_link">
-    <inertial>
-      <mass value="0.03"/>
-      <inertia ixx="0.00003" ixy="0" ixz="0" iyy="0.00003" iyz="0" izz="0.00003"/>
-    </inertial>
-    <collision>
-      <geometry><sphere radius="${caster_radius}"/></geometry>
-      <surface>
-        <friction>
-          <ode>
-            <mu>0.000001</mu>
-            <mu2>0.000001</mu2>
-            <slip1>1.0</slip1>
-            <slip2>1.0</slip2>
-          </ode>
-        </friction>
-        <contact>
-          <ode><kp>80000</kp><kd>0.5</kd><max_vel>0.1</max_vel><min_depth>0.0005</min_depth></ode>
-        </contact>
-      </surface>
-    </collision>
-    <visual>
-      <geometry><sphere radius="${caster_radius}"/></geometry>
-      <material name="rim_gray"/>
-    </visual>
-  </link>
-  <joint name="front_caster_joint" type="fixed">
-    <parent link="base_link"/>
-    <child link="front_caster_link"/>
-    <origin xyz="0.19 0 ${caster_z}" rpy="0 0 0"/>
-  </joint>
-  <link name="rear_caster_link">
-    <inertial>
-      <mass value="0.03"/>
-      <inertia ixx="0.00003" ixy="0" ixz="0" iyy="0.00003" iyz="0" izz="0.00003"/>
-    </inertial>
-    <collision>
-      <geometry><sphere radius="${caster_radius}"/></geometry>
-      <surface>
-        <friction>
-          <ode>
-            <mu>0.000001</mu>
-            <mu2>0.000001</mu2>
-            <slip1>1.0</slip1>
-            <slip2>1.0</slip2>
-          </ode>
-        </friction>
-        <contact>
-          <ode><kp>80000</kp><kd>0.5</kd><max_vel>0.1</max_vel><min_depth>0.0005</min_depth></ode>
-        </contact>
-      </surface>
-    </collision>
-    <visual>
-      <geometry><sphere radius="${caster_radius}"/></geometry>
-      <material name="rim_gray"/>
-    </visual>
-  </link>
-  <joint name="rear_caster_joint" type="fixed">
-    <parent link="base_link"/>
-    <child link="rear_caster_link"/>
-    <origin xyz="-0.19 0 ${caster_z}" rpy="0 0 0"/>
   </joint>
   <link name="sensor_mast_link">

Commit message: Add visual-only support wheels

File: src/diffbot_gazebo/urdf/diffbot.urdf.xacro (robot description, xacro)
@@ -10,4 +10,6 @@
   <xacro:property name="wheel_z" value="0.085"/>
   <xacro:property name="base_origin_z" value="${base_height / 2.0 + 0.035}"/>
+  <xacro:property name="support_ball_radius" value="0.022"/>
+  <xacro:property name="support_ball_z" value="${support_ball_radius - base_origin_z + 0.004}"/>
   <material name="body_blue"><color rgba="0.05 0.22 0.55 1"/></material>
   <material name="top_silver"><color rgba="0.75 0.8 0.86 1"/></material>
@@ -124,4 +126,26 @@
     <origin xyz="${wheel_x} ${-wheel_y} ${-base_height / 2.0 + wheel_z - 0.035}" rpy="0 0 0"/>
     <axis xyz="0 1 0"/>
+  </joint>
+  <link name="front_visual_support_ball_link">
+    <visual>
+      <geometry><sphere radius="${support_ball_radius}"/></geometry>
+      <material name="rim_gray"/>
+    </visual>
+  </link>
+  <joint name="front_visual_support_ball_joint" type="fixed">
+    <parent link="base_link"/>
+    <child link="front_visual_support_ball_link"/>
+    <origin xyz="0.19 0 ${support_ball_z}" rpy="0 0 0"/>
+  </joint>
+  <link name="rear_visual_support_ball_link">
+    <visual>
+      <geometry><sphere radius="${support_ball_radius}"/></geometry>
+      <material name="rim_gray"/>
+    </visual>
+  </link>
+  <joint name="rear_visual_support_ball_joint" type="fixed">
+    <parent link="base_link"/>
+    <child link="rear_visual_support_ball_link"/>
+    <origin xyz="-0.19 0 ${support_ball_z}" rpy="0 0 0"/>
   </joint>
   <link name="sensor_mast_link">
