Commit message: Stabilize support balls without lifting drive wheels

File: src/diffbot_gazebo/urdf/diffbot.urdf.xacro (robot description, xacro)
@@ -11,5 +11,5 @@
   <xacro:property name="base_origin_z" value="${base_height / 2.0 + 0.035}"/>
   <xacro:property name="support_ball_radius" value="0.022"/>
-  <xacro:property name="support_ball_z" value="${support_ball_radius - base_origin_z + 0.004}"/>
+  <xacro:property name="support_ball_z" value="${support_ball_radius - base_origin_z + 0.001}"/>
   <material name="body_blue"><color rgba="0.05 0.22 0.55 1"/></material>
   <material name="top_silver"><color rgba="0.75 0.8 0.86 1"/></material>
@@ -128,4 +128,25 @@
   </joint>
   <link name="front_visual_support_ball_link">
+    <collision>
+      <geometry><sphere radius="${support_ball_radius}"/></geometry>
+      <surface>
+        <friction>
+          <ode>
+            <mu>0.000001</mu>
+            <mu2>0.000001</mu2>
+            <slip1>1.0</slip1>
+            <slip2>1.0</slip2>
+          </ode>
+        </friction>
+        <contact>
+          <ode>
+            <kp>60000</kp>
+            <kd>0.3</kd>
+            <max_vel>0.05</max_vel>
+            <min_depth>0.0002</min_depth>
+          </ode>
+        </contact>
+      </surface>
+    </collision>
     <visual>
       <geometry><sphere radius="${support_ball_radius}"/></geometry>
@@ -139,4 +160,25 @@
   </joint>
   <link name="rear_visual_support_ball_link">
+    <collision>
+      <geometry><sphere radius="${support_ball_radius}"/></geometry>
+      <surface>
+        <friction>
+          <ode>
+            <mu>0.000001</mu>
+            <mu2>0.000001</mu2>
+            <slip1>1.0</slip1>
+            <slip2>1.0</slip2>
+          </ode>
+        </friction>
+        <contact>
+          <ode>
+            <kp>60000</kp>
+            <kd>0.3</kd>
+            <max_vel>0.05</max_vel>
+            <min_depth>0.0002</min_depth>
+          </ode>
+        </contact>
+      </surface>
+    </collision>
     <visual>
       <geometry><sphere radius="${support_ball_radius}"/></geometry>
